File: electronics/view_base/view_base.kicad_sch (KiCad schematic)
At the start: 107 parts, among them J1 BLDC, J2 USB_C_Receptacle_USB2.0, J3 LCD, J4 A, J5 B, Q1 MMBT4403, Q2 UMH3N, U1 MT6701-CT, U2 T-Micro32_Plus, U3 CH340C, U4 HX711, U5 TMC6300, U6 AP2114HA-3.3, U7 SN74LV1T34DBV, U8 VEML7700, U9 TS1117BCW33_RPG

Commit message: Use ESP32-S3-MINI-1 in place of TMicro32 Plus
Parts:
- removed C28: 1uF, Capacitor_SMD:C_0603_1608Metric, symbol Device:C_Small
- removed Q2: UMH3N, Package_TO_SOT_SMD:SOT-363_SC-70-6, symbol Transistor_BJT:UMH3N
- removed U2: T-Micro32_Plus, lilygo_micro32:T-Micro32, symbol lilygo_micro32:T-Micro32_Plus
- removed U3: CH340C, Package_SO:SOIC-16_3.9x9.9mm_P1.27mm, symbol Interface_USB:CH340C
- added D9: NUF2042XV6T1G, Package_TO_SOT_SMD:SOT-563, symbol NUF2042XV6T1G:NUF2042XV6T1G
- added SW1, SW2: SW_Push, Button_Switch_SMD:SW_SPST_B3U-3000P-B, symbol Switch:SW_Push
- added TP17: MTMS, Modified:TestPoint_Pad_D2.0mm_ValueSilk, symbol Connector:TestPoint_Small
- added TP18: MTDI, Modified:TestPoint_Pad_D2.0mm_ValueSilk, symbol Connector:TestPoint_Small
- added TP19: MTDO, Modified:TestPoint_Pad_D2.0mm_ValueSilk, symbol Connector:TestPoint_Small
- added TP20: MTCK, Modified:TestPoint_Pad_D2.0mm_ValueSilk, symbol Connector:TestPoint_Small
- added TP21: IO8, Modified:TestPoint_Pad_D2.0mm_ValueSilk, symbol Connector:TestPoint_Small
- added TP22: IO9, Modified:TestPoint_Pad_D2.0mm_ValueSilk, symbol Connector:TestPoint_Small
- added TP23: IO10, Modified:TestPoint_Pad_D2.0mm_ValueSilk, symbol Connector:TestPoint_Small
- added TP24: IO11, Modified:TestPoint_Pad_D2.0mm_ValueSilk, symbol Connector:TestPoint_Small
- added TP25: IO16, Modified:TestPoint_Pad_D2.0mm_ValueSilk, symbol Connector:TestPoint_Small
- added TP26: IO17, Modified:TestPoint_Pad_D2.0mm_ValueSilk, symbol Connector:TestPoint_Small
- added TP27: IO18, Modified:TestPoint_Pad_D2.0mm_ValueSilk, symbol Connector:TestPoint_Small
- added U2: ESP32-S3-MINI-1, PCM_Espressif:ESP32-S3-MINI-1, symbol PCM_Espressif:ESP32-S3-MINI-1
- C11: value 0.1uF -> 1uF; Digikey 1276-1935-1-ND -> 1276-1102-1-ND; LCSC C1591 -> C5673; Mouser 187-CL10B104KB8NNWC -> 187-CL10A105KA8NNNC
- C24: value 10uF -> 22uF; Digikey 1276-2891-1-ND -> 1276-CL21A226MAYNNNECT-ND; LCSC C2922480 -> C98190; Mouser 187-CL21A106KAYNNNE -> 187-CL21A226MAYNNNE
Connections:
- net +3V3: now also U2.3 (3V3); no longer C11.1
- net +5V: now also D9.5 (VBUS)
- net ESP32_BOOT: now also SW2.1, U2.4 (IO0)
- net ESP32_EN: now also C11.1, SW1.1, U2.45 (EN)
- net GND: now also D9.2 (GND), SW1.2, SW2.2, U2.1 (GND), U2.2 (GND), U2.42 (GND), U2.43 (GND), U2.46 (GND), U2.47 (GND), U2.48 (GND), U2.49 (GND), U2.50 (GND), U2.51 (GND), U2.52 (GND), U2.53 (GND), U2.54 (GND), U2.55 (GND), U2.56 (GND), U2.57 (GND), U2.58 (GND), U2.59 (GND), U2.60 (GND), U2.61 (GND), U2.62 (GND), U2.63 (GND), U2.64 (GND), U2.65 (GND)
- net LCD_BACKLIGHT: now also U2.34 (IO38)
- net LCD_CMD: now also U2.30 (IO48)
- net LCD_CS: now also U2.29 (IO34)
- net LCD_DATA: now also U2.31 (IO35)
- net LCD_RST: now also U2.33 (IO37)
- net LCD_SCK: now also U2.32 (IO36)
- net LED_DATA_3V3: now also U2.19 (IO15)
- net MAG_CLK: now also U2.17 (IO13)
- net MAG_CSN: now also U2.16 (IO12)
- net MAG_DO: now also U2.18 (IO14)
- net SCL: now also U2.27 (IO47)
- net SDA: now also U2.28 (IO33)
- net STRAIN_DO: now also U2.25 (IO21)
- net STRAIN_SCK: now also U2.26 (IO26)
- net TMC_DIAG: now also U2.5 (IO1)
- net TMC_UH: now also U2.9 (IO5)
- net TMC_UL: now also U2.8 (IO4)
- net TMC_VH: now also U2.10 (IO6)
- net TMC_VL: now also U2.6 (IO2)
- net TMC_WH: now also U2.11 (IO7)
- net TMC_WL: now also U2.7 (IO3)
- net USB_D+: now also D9.3 (D2(I))
- net USB_D-: now also D9.1 (D1(I))
- net USB_SERIAL_RXI renamed U0TXD
- net U0TXD: now also U2.39 (IO43)
- net USB_SERIAL_TXO renamed U0RXD
- net U0RXD: now also U2.40 (IO44)
- new net IO10: TP23.1, U2.14 (IO10)
- new net IO11: TP24.1, U2.15 (IO11)
- new net IO16: TP25.1, U2.20 (IO16)
- new net IO17: TP26.1, U2.21 (IO17)
- new net IO18: TP27.1, U2.22 (IO18)
- new net IO8: TP21.1, U2.12 (IO8)
- new net IO9: TP22.1, U2.13 (IO9)
- new net JTAG_MTCK: TP20.1, U2.35 (IO39)
- new net JTAG_MTDI: TP18.1, U2.37 (IO41)
- new net JTAG_MTDO: TP19.1, U2.36 (IO40)
- new net JTAG_MTMS: TP17.1, U2.38 (IO42)
- new net MCU_USB_D+: D9.4 (D2(0)), U2.24 (IO20)
- new net MCU_USB_D-: D9.6 (D1(0)), U2.23 (IO19)
- no-connect marks 24 -> 17
Other:
- note added: "MCU - ESP32 (ESP32-S3-WROOM-2)"
- note added: "Reset/Boot via push switch"
- note added: "TVS for ESD protection"
- note removed: "GPIO12=MTDI. Should be 0 on boot for 3.3v built-in flash/psram on ESP32-PICO-v3-02"
- note removed: "IO2 must be 0 to enter UART download mode"
- note removed: "MCU - ESP32 (T-MICRO32 PLUS)"
- note removed: "Reset/Boot via USB serial"
- moved on the sheet: TP13, TP14
